Commit message: [feat] 补充3d模型

File: pc/ros2_ws/src/arm_description/urdf/arm_platform.urdf.xacro (robot description, xacro)
@@ -2,123 +2,117 @@
 <robot xmlns:xacro="http://www.ros.org/wiki/xacro" name="arm_platform">
   <xacro:property name="pi_const" value="3.1415926535897931"/>
-  <xacro:property name="base_height" value="0.06"/>
-  <xacro:property name="link_1_length" value="0.08"/>
-  <xacro:property name="link_2_length" value="0.10"/>
-  <xacro:property name="link_3_length" value="0.10"/>
-  <xacro:property name="link_4_length" value="0.08"/>
-  <xacro:property name="link_5_length" value="0.05"/>
-  <xacro:property name="link_radius" value="0.015"/>
-  <material name="base_blue">
-    <color rgba="0.18 0.31 0.45 1.0"/>
+  <xacro:property name="joint_limit" value="${pi_const / 2.0}"/>
+  <xacro:property name="mesh_scale" value="0.001 0.001 0.001"/>
+  <!-- Dimensions are derived from the STL bounding boxes, converted from millimetres. -->
+  <xacro:property name="base_turntable_x" value="0.0"/>
+  <xacro:property name="base_turntable_y" value="0.0"/>
+  <xacro:property name="base_kasa_z" value="0.01"/>
+  <xacro:property name="base_rotate_height" value="0.08"/>
+  <xacro:property name="base_govde_z" value="0.01"/>
+  <xacro:property name="base_to_shoulder_x" value="0.04"/>
+  <xacro:property name="base_to_shoulder_y" value="0.0"/>
+  <xacro:property name="base_to_shoulder_height" value="0.04"/>
+  <xacro:property name="upper_arm_length" value="0.1985"/>
+  <xacro:property name="upper_arm_elbow_z_offset" value="-0.038"/>
+  <xacro:property name="forearm_zero_pitch" value="1.3962634015954636"/>
+  <xacro:property name="forearm_near_hole_x" value="0.0"/>
+  <xacro:property name="forearm_far_hole_x" value="-0.135"/>
+  <xacro:property name="forearm_length" value="${forearm_near_hole_x - forearm_far_hole_x}"/>
+  <xacro:property name="wrist_mesh_x" value="0.0"/>
+  <xacro:property name="wrist_to_hand" value="0.043"/>
+  <xacro:property name="hand_mesh_x" value="0.0"/>
+  <xacro:property name="hand_to_tool" value="0.05"/>
+  <material name="printed_teal">
+    <color rgba="0.10 0.42 0.48 1.0"/>
   </material>
-  <material name="arm_orange">
-    <color rgba="0.83 0.48 0.21 1.0"/>
+  <material name="printed_orange">
+    <color rgba="0.86 0.46 0.18 1.0"/>
   </material>
-  <material name="joint_dark">
-    <color rgba="0.15 0.15 0.15 1.0"/>
+  <material name="printed_lime">
+    <color rgba="0.46 0.63 0.20 1.0"/>
   </material>
+  <material name="hardware_dark">
+    <color rgba="0.12 0.12 0.13 1.0"/>
+  </material>
+  <material name="gear_yellow">
+    <color rgba="0.95 0.70 0.20 1.0"/>
+  </material>
+  <xacro:macro name="mesh_visual" params="filename xyz:='0 0 0' rpy:='0 0 0' material:='printed_orange'">
+    <visual>
+      <origin xyz="${xyz}" rpy="${rpy}"/>
+      <geometry>
+        <mesh filename="package://arm_description/meshes/${filename}" scale="${mesh_scale}"/>
+      </geometry>
+      <material name="${material}"/>
+    </visual>
+  </xacro:macro>
   <link name="base_link">
-    <visual>
-      <geometry>
-        <cylinder radius="0.05" length="${base_height}"/>
-      </geometry>
-      <material name="base_blue"/>
-    </visual>
+    <xacro:mesh_visual filename="Alt_Kasa.stl" xyz="${base_turntable_x} ${base_turntable_y} ${base_kasa_z}" material="printed_teal"/>
   </link>
   <link name="link_1">
-    <visual>
-      <origin xyz="0 0 ${link_1_length / 2.0}" rpy="0 0 0"/>
-      <geometry>
-        <cylinder radius="${link_radius}" length="${link_1_length}"/>
-      </geometry>
-      <material name="joint_dark"/>
-    </visual>
+    <xacro:mesh_visual filename="Alt_Govde.stl" xyz="0 0 ${base_govde_z}" material="printed_lime"/>
   </link>
   <joint name="joint_1" type="revolute">
     <parent link="base_link"/>
     <child link="link_1"/>
-    <origin xyz="0 0 ${base_height / 2.0}" rpy="0 0 0"/>
+    <origin xyz="${base_turntable_x} ${base_turntable_y} ${base_rotate_height}" rpy="0 0 0"/>
     <axis xyz="0 0 1"/>
-    <limit lower="${-pi}" upper="${pi}" effort="1.0" velocity="0.5"/>
+    <limit lower="${-joint_limit}" upper="${joint_limit}" effort="1.0" velocity="0.5"/>
   </joint>
   <link name="link_2">
-    <visual>
-        <origin xyz="${link_2_length / 2.0} 0 0" rpy="0 ${pi_const / 2.0} 0"/>
-      <geometry>
-        <cylinder radius="${link_radius}" length="${link_2_length}"/>
-      </geometry>
-      <material name="arm_orange"/>
-    </visual>
+    <xacro:mesh_visual filename="Alt_Kol.stl" xyz="0.1039 0 0" rpy="0 ${pi_const / 2.0} 0" material="printed_orange"/>
   </link>
   <joint name="joint_2" type="revolute">
     <parent link="link_1"/>
     <child link="link_2"/>
-    <origin xyz="0 0 ${link_1_length}" rpy="0 0 0"/>
+    <origin xyz="${base_to_shoulder_x} ${base_to_shoulder_y} ${base_to_shoulder_height}" rpy="0 ${-pi_const / 2.0} 0"/>
     <axis xyz="0 1 0"/>
-    <limit lower="${-pi_const}" upper="${pi_const}" effort="1.0" velocity="0.5"/>
+    <limit lower="${-joint_limit}" upper="${joint_limit}" effort="1.0" velocity="0.5"/>
   </joint>
   <link name="link_3">
-    <visual>
-        <origin xyz="${link_3_length / 2.0} 0 0" rpy="0 ${pi_const / 2.0} 0"/>
-      <geometry>
-        <cylinder radius="${link_radius}" length="${link_3_length}"/>
-      </geometry>
-      <material name="arm_orange"/>
-    </visual>
+    <xacro:mesh_visual filename="On_Kol.stl" xyz="${forearm_near_hole_x} 0 0" rpy="0 0 ${pi_const}" material="printed_orange"/>
   </link>
   <joint name="joint_3" type="revolute">
     <parent link="link_2"/>
     <child link="link_3"/>
-    <origin xyz="${link_2_length} 0 0" rpy="0 0 0"/>
+    <origin xyz="${upper_arm_length} 0 ${upper_arm_elbow_z_offset}" rpy="0 ${forearm_zero_pitch} 0"/>
     <axis xyz="0 1 0"/>
-    <limit lower="${-pi_const}" upper="${pi_const}" effort="1.0" velocity="0.5"/>
+    <limit lower="${-joint_limit}" upper="${joint_limit}" effort="1.0" velocity="0.5"/>
   </joint>
   <link name="link_4">
-    <visual>
-        <origin xyz="${link_4_length / 2.0} 0 0" rpy="0 ${pi_const / 2.0} 0"/>
-      <geometry>
-        <cylinder radius="${link_radius}" length="${link_4_length}"/>
-      </geometry>
-      <material name="joint_dark"/>
-    </visual>
+    <xacro:mesh_visual filename="Bilek.stl" xyz="${wrist_mesh_x} 0 0" rpy="0 ${pi_const / 2.0} 0" material="printed_lime"/>
   </link>
   <joint name="joint_4" type="revolute">
     <parent link="link_3"/>
     <child link="link_4"/>
-    <origin xyz="${link_3_length} 0 0" rpy="0 0 0"/>
+    <origin xyz="${forearm_length} 0 0" rpy="0 0 0"/>
     <axis xyz="0 1 0"/>
-    <limit lower="${-pi_const}" upper="${pi_const}" effort="1.0" velocity="0.5"/>
+    <limit lower="${-joint_limit}" upper="${joint_limit}" effort="1.0" velocity="0.5"/>
   </joint>
   <link name="link_5">
-    <visual>
-      <origin xyz="0 0 ${link_5_length / 2.0}" rpy="0 0 0"/>
-      <geometry>
-        <cylinder radius="${link_radius * 0.8}" length="${link_5_length}"/>
-      </geometry>
-      <material name="arm_orange"/>
-    </visual>
+    <xacro:mesh_visual filename="El.stl" xyz="${hand_mesh_x} 0 0" rpy="0 ${pi_const / 2.0} 0" material="printed_teal"/>
+    <xacro:mesh_visual filename="El_Ust.stl" xyz="${hand_mesh_x} 0 0" rpy="0 ${pi_const / 2.0} 0" material="printed_lime"/>
   </link>
   <joint name="joint_5" type="revolute">
     <parent link="link_4"/>
     <child link="link_5"/>
-    <origin xyz="${link_4_length} 0 0" rpy="0 0 0"/>
+    <origin xyz="${wrist_to_hand} 0 0" rpy="0 0 0"/>
     <axis xyz="1 0 0"/>
-    <limit lower="${-pi_const}" upper="${pi_const}" effort="1.0" velocity="0.5"/>
+    <limit lower="${-joint_limit}" upper="${joint_limit}" effort="1.0" velocity="0.5"/>
   </joint>
   <link name="tool_link">
-    <visual>
-      <origin xyz="0 0 ${link_5_length / 2.0}" rpy="0 0 0"/>
-      <geometry>
-        <box size="0.03 0.03 ${link_5_length}"/>
-      </geometry>
-      <material name="joint_dark"/>
-    </visual>
+    <xacro:mesh_visual filename="Parmak_Disli_X_2.stl" xyz="${hand_to_tool} 0.018 0" rpy="${pi_const} 0 0" material="gear_yellow"/>
+    <xacro:mesh_visual filename="Parmak_X_2.stl" xyz="${hand_to_tool + 0.022} 0.018 0" rpy="${pi_const} 0 0" material="printed_orange"/>
+    <xacro:mesh_visual filename="Parmak_2_X_2.stl" xyz="${hand_to_tool + 0.045} 0.018 -0.0025" rpy="${pi_const} 0 0" material="printed_lime"/>
+    <xacro:mesh_visual filename="Parmak_Disli_X_2.stl" xyz="${hand_to_tool} -0.018 0" material="gear_yellow"/>
+    <xacro:mesh_visual filename="Parmak_X_2.stl" xyz="${hand_to_tool + 0.022} -0.018 0" material="printed_orange"/>
+    <xacro:mesh_visual filename="Parmak_2_X_2.stl" xyz="${hand_to_tool + 0.045} -0.018 -0.0025" material="printed_lime"/>
   </link>
   <joint name="joint_6" type="revolute">
     <parent link="link_5"/>
     <child link="tool_link"/>
-    <origin xyz="0 0 ${link_5_length}" rpy="0 0 0"/>
+    <origin xyz="${hand_to_tool} 0 0" rpy="0 0 0"/>
     <axis xyz="0 0 1"/>
-    <limit lower="${-pi}" upper="${pi}" effort="1.0" velocity="0.5"/>
+    <limit lower="${-joint_limit}" upper="${joint_limit}" effort="1.0" velocity="0.5"/>
   </joint>
 </robot>
